Commit message: Put base_link on correct height wrt floor and add initial guess for laser_link

File: neato_description/urdf/neato.urdf.xacro (robot description, xacro)
@@ -1,7 +1,14 @@
 <?xml version="1.0"?>
 <robot xmlns:xacro="http://ros.org/wiki/xacro" name="neato">
+  <link name="base_footprint">
+  </link>
+  <joint name="footprint_to_link" type="fixed">
+    <parent link="base_footprint"/>
+    <child link="base_link"/>
+    <origin xyz="0 0 0.02" rpy="0 0 0" />
+  </joint>
   <link name="base_link">
     <visual>
-      <origin xyz="0.150 -0.165 -0.040" rpy="0 0 1.57" />
+      <origin xyz="0.150 -0.165 0" rpy="0 0 1.57" />
       <geometry>
         <mesh filename="package://neato_description/meshes/neato.dae" scale="0.025 0.025 0.025"/>
@@ -9,3 +16,9 @@
     </visual>
   </link>
+  <joint name="base_to_laser" type="fixed">
+    <parent link="base_link"/>
+    <child link="laser_link"/>
+    <origin xyz="-0.1 0 0.083" rpy="0 0 0" />
+  </joint>
+  <link name="laser_link"/>
 </robot>

Commit message: Add two wheels. The baselink mesh is not entirely accurate yet but it'll do

File: neato_description/urdf/neato.urdf.xacro (robot description, xacro)
@@ -1,4 +1,23 @@
 <?xml version="1.0"?>
 <robot xmlns:xacro="http://ros.org/wiki/xacro" name="neato">
+  <xacro:macro name="wheel" params="side">
+    <link name="${side}_wheel_link">
+    <visual>
+      <origin xyz="0 0 0" rpy="0 0 0" />
+      <geometry>
+        <cylinder radius="0.0365" length="0.014"/>
+      </geometry>
+      <material name="Rubber">
+        <color rgba="0 0 0 1"/>
+      </material>
+    </visual>
+    <collision>
+      <origin xyz="0 0 0" rpy="0 0 0"/>
+      <geometry>
+        <cylinder radius="0.0365" length="0.014"/>
+      </geometry>
+    </collision>
+  </link>
+  </xacro:macro>
   <link name="base_footprint">
   </link>
@@ -22,3 +41,15 @@
   </joint>
   <link name="laser_link"/>
+  <joint name="base_to_left_wheel" type="fixed">
+    <parent link="base_link"/>
+    <child link="left_wheel_link"/>
+    <origin xyz="0 ${0.243 / 2} 0.016" rpy="1.57 0 0" /> <!--wheel-to-wheel distance/2-->
+  </joint>
+  <joint name="base_to_right_wheel" type="fixed">
+    <parent link="base_link"/>
+    <child link="right_wheel_link"/>
+    <origin xyz="0 -${0.243 / 2} 0.016" rpy="1.57 0 0" />
+  </joint>
+  <xacro:wheel side="left"/>
+  <xacro:wheel side="right"/>
 </robot>

Commit message: Using my own custom mesh
from https://cad.onshape.com/documents/274eac952e0f9663ef5ae2ad/w/975287c2a5d4f4815380c41d/e/d8426bc7f59956a42e4edbd6, measured with a tape measure and caliper

File: neato_description/urdf/neato.urdf.xacro (robot description, xacro)
@@ -29,14 +29,14 @@
   <link name="base_link">
     <visual>
-      <origin xyz="0.150 -0.165 0" rpy="0 0 1.57" />
+      <origin xyz="0 0 0" rpy="0 0 1.57" />
       <geometry>
-        <mesh filename="package://neato_description/meshes/neato.dae" scale="0.025 0.025 0.025"/>
+        <mesh filename="package://neato_description/meshes/NeatoDSeries.dae" />
       </geometry>
     </visual>
   </link>
   <joint name="base_to_laser" type="fixed">
-    <parent link="base_link"/>
+    <parent link="base_footprint"/>
     <child link="laser_link"/>
-    <origin xyz="-0.1 0 0.083" rpy="0 0 0" />
+    <origin xyz="-0.1 0 0.0825" rpy="0 0 0" />
   </joint>
   <link name="laser_link"/>
